File: Gyroscope.kicad_pcb (KiCad board)
At the start: 2 copper layers, 5 parts, among them U1 IIS3DWB, U2 APS6404L-3SQRx-SN, U3 STM32G431C6Tx, U4 W25Q128JVS, U5 CR2013-MI2120

Commit message: refresh
Parts:
- added J1: Barrel_Jack_Switch, Connector_BarrelJack:BarrelJack_GCT_DCJ200-10-A_Horizontal, F.Cu at (109.9, 96.2)
- added J2: Micro_SD_Card_Det2, Connector_Card:microSD_HC_Hirose_DM3AT-SF-PEJM5, F.Cu at (95.9, 103.5)
- added U6: AP2112K-3.3, Package_TO_SOT_SMD:SOT-23-5, F.Cu at (130.6, 106.9)
- added U7: 74LVC1G139, Package_SO:VSSOP-8_2.3x2mm_P0.5mm, F.Cu at (130.8, 102.7)
- moved U5 21.3 mm to (90.2, 63.2)
- moved U3 10.6 mm to (122.4, 99.9)
- moved U2 6.28 mm to (132.3, 97.6)
- moved U4 5.94 mm to (121.9, 109.1)
- moved U1 2.84 mm to (130.7, 111.1)
Connections:
- U1 pad 1: unconnected-(U1-SDO-Pad1) -> Net-(U1-SDO)
- U1 pad 12: unconnected-(U1-CS-Pad12) -> Net-(U1-CS)
- U1 pad 13: unconnected-(U1-SPC-Pad13) -> Net-(U1-SPC)
- U1 pad 14: unconnected-(U1-SDI-Pad14) -> Net-(U1-SDI)
- U1 pad 2: Net-(U1-GND-Pad2) -> GND
- U1 pad 3: Net-(U1-GND-Pad2) -> GND
- U1 pad 4: unconnected-(U1-INT1-Pad4) -> Net-(U1-INT1)
- U1 pad 5: unconnected-(U1-VDD_IO-Pad5) -> Net-(U1-VDD)
- U1 pad 6: Net-(U1-GND-Pad2) -> GND
- U1 pad 7: Net-(U1-GND-Pad2) -> GND
- U1 pad 8: unconnected-(U1-VDD-Pad8) -> Net-(U1-VDD)
- U1 pad 9: unconnected-(U1-INT2-Pad9) -> Net-(U1-INT2)
- U2 pad 1: unconnected-(U2-~{CE}-Pad1) -> Net-(U2-~{CE})
- U2 pad 2: unconnected-(U2-SO/SIO1-Pad2) -> Net-(U2-SO/SIO1)
- U2 pad 3: unconnected-(U2-SIO2-Pad3) -> Net-(U2-SIO2)
- U2 pad 4: unconnected-(U2-VSS-Pad4) -> GND
- U2 pad 5: unconnected-(U2-SI/SIO0-Pad5) -> Net-(U2-SI/SIO0)
- U2 pad 6: unconnected-(U2-SCLK-Pad6) -> Net-(U2-SCLK)
- U2 pad 7: unconnected-(U2-SIO3-Pad7) -> Net-(U2-SIO2)
- U2 pad 8: unconnected-(U2-VDD-Pad8) -> +3.3V
- U3 pad 1: unconnected-(U3-VBAT-Pad1) -> +3.3V
- U3 pad 12: unconnected-(U3-PA4-Pad12) -> Net-(U3-PA4)
- U3 pad 13: unconnected-(U3-PA5-Pad13) -> Net-(U3-PA5)
- U3 pad 14: unconnected-(U3-PA6-Pad14) -> Net-(U3-PA6)
- U3 pad 15: unconnected-(U3-PA7-Pad15) -> Net-(U3-PA7)
- U3 pad 19: unconnected-(U3-VSSA-Pad19) -> GND
- U3 pad 21: unconnected-(U3-VDDA-Pad21) -> Net-(U3-VDDA)
- U3 pad 23: Net-(U3-VSS-Pad23) -> GND
- U3 pad 24: unconnected-(U3-VDD-Pad24) -> +3.3V
- U3 pad 26: unconnected-(U3-PB12-Pad26) -> Net-(U2-~{CE})
- U3 pad 27: unconnected-(U3-PB13-Pad27) -> Net-(U2-SCLK)
- U3 pad 28: unconnected-(U3-PB14-Pad28) -> Net-(U2-SO/SIO1)
- U3 pad 29: unconnected-(U3-PB15-Pad29) -> Net-(U2-SI/SIO0)
- U3 pad 32: unconnected-(U3-PA10-Pad32) -> Net-(U3-PA10)
- U3 pad 33: unconnected-(U3-PA11-Pad33) -> Net-(U3-PA11)
- U3 pad 34: unconnected-(U3-PA12-Pad34) -> Net-(U3-PA12)
- U3 pad 35: Net-(U3-VSS-Pad23) -> GND
- U3 pad 36: unconnected-(U3-VDD-Pad36) -> +3.3V
- U3 pad 37: unconnected-(U3-PA13-Pad37) -> Net-(U1-INT2)
- U3 pad 38: unconnected-(U3-PA14-Pad38) -> Net-(U1-INT1)
- U3 pad 39: unconnected-(U3-PA15-Pad39) -> Net-(U1-CS)
- U3 pad 40: unconnected-(U3-PB3-Pad40) -> Net-(U1-SDO)
- U3 pad 41: unconnected-(U3-PB4-Pad41) -> Net-(U1-SDI)
- U3 pad 42: unconnected-(U3-PB5-Pad42) -> Net-(U1-SPC)
- U3 pad 47: Net-(U3-VSS-Pad23) -> GND
- U3 pad 48: unconnected-(U3-VDD-Pad48) -> +3.3V
- U4 pad 1: unconnected-(U4-~{CS}-Pad1) -> Net-(U3-PA4)
- U4 pad 2: unconnected-(U4-DO/IO_{1}-Pad2) -> Net-(U3-PA6)
- U4 pad 3: unconnected-(U4-~{WP}/IO_{2}-Pad3) -> Net-(U4-~{HOLD}/~{RESET}/IO_{3})
- U4 pad 4: unconnected-(U4-GND-Pad4) -> GND
- U4 pad 5: unconnected-(U4-DI/IO_{0}-Pad5) -> Net-(U3-PA7)
- U4 pad 6: unconnected-(U4-CLK-Pad6) -> Net-(U3-PA5)
- U4 pad 7: unconnected-(U4-~{HOLD}/~{RESET}/IO_{3}-Pad7) -> Net-(U4-~{HOLD}/~{RESET}/IO_{3})
- U4 pad 8: unconnected-(U4-VCC-Pad8) -> +3.3V
- U5 pad 2: unconnected-(U5-GND-Pad2) -> GND
- U5 pad 3: unconnected-(U5-~{CS}-Pad3) -> Net-(U3-PA12)
- U5 pad 6: unconnected-(U5-MOSI-Pad6) -> Net-(U3-PA11)
- U5 pad 9: unconnected-(U5-MISO-Pad9) -> Net-(U3-PA10)

Commit message: refresh
Parts:
- added C10: 1u, Capacitor_SMD:C_0805_2012Metric, F.Cu at (157.6, 119.5)
- added C11: 100n, Capacitor_SMD:C_0402_1005Metric, F.Cu at (159.7, 110.1)
- added C12: 100n, Capacitor_SMD:C_0402_1005Metric, F.Cu at (159.7, 112.1)
- added C13: 100n, Capacitor_SMD:C_0402_1005Metric, F.Cu at (159.7, 114.0)
- added C14: 100n, Capacitor_SMD:C_0402_1005Metric, F.Cu at (162.5, 110.1)
- added C15: 100n, Capacitor_SMD:C_0402_1005Metric, F.Cu at (162.5, 112.1)
- added C16: 100n, Capacitor_SMD:C_0402_1005Metric, F.Cu at (162.5, 114.0)
- added C6: 100n, Capacitor_SMD:C_0402_1005Metric, F.Cu at (156.8, 110.1)
- added C7: 100n, Capacitor_SMD:C_0402_1005Metric, F.Cu at (156.8, 112.1)
- added C8: 1u, Capacitor_SMD:C_0805_2012Metric, F.Cu at (157.6, 116.5)
- added C9: 100n, Capacitor_SMD:C_0402_1005Metric, F.Cu at (156.8, 114.0)
- added H1: MountingScrew, MountingHole:MountingHole_2.2mm_M2_DIN965_Pad_TopBottom, F.Cu at (152.7, 111.8)
- added H2: MountingScrew, MountingHole:MountingHole_2.2mm_M2_DIN965_Pad_TopBottom, F.Cu at (152.7, 117.1)
- added H3: MountingScrew, MountingHole:MountingHole_2.2mm_M2_DIN965_Pad_TopBottom, F.Cu at (152.7, 122.5)
- added H4: MountingScrew, MountingHole:MountingHole_2.2mm_M2_DIN965_Pad_TopBottom, F.Cu at (152.7, 127.8)
Connections:
- U1 pad 1: Net-(U1-SDO) -> unconnected-(U1-SDO-Pad1)
- U1 pad 12: Net-(U1-CS) -> unconnected-(U1-CS-Pad12)
- U1 pad 13: Net-(U1-SPC) -> unconnected-(U1-SPC-Pad13)
- U1 pad 14: Net-(U1-SDI) -> unconnected-(U1-SDI-Pad14)
- U1 pad 2: GND -> Net-(U1-GND-Pad2)
- U1 pad 3: GND -> Net-(U1-GND-Pad2)
- U1 pad 4: Net-(U1-INT1) -> unconnected-(U1-INT1-Pad4)
- U1 pad 6: GND -> Net-(U1-GND-Pad2)
- U1 pad 7: GND -> Net-(U1-GND-Pad2)
- U1 pad 9: Net-(U1-INT2) -> unconnected-(U1-INT2-Pad9)
- U2 pad 1: Net-(U2-~{CE}) -> unconnected-(U2-~{CE}-Pad1)
- U2 pad 2: Net-(U2-SO/SIO1) -> unconnected-(U2-SO/SIO1-Pad2)
- U2 pad 3: Net-(U2-SIO2) -> unconnected-(U2-SIO2-Pad3)
- U2 pad 4: GND -> unconnected-(U2-VSS-Pad4)
- U2 pad 5: Net-(U2-SI/SIO0) -> unconnected-(U2-SI/SIO0-Pad5)
- U2 pad 6: Net-(U2-SCLK) -> unconnected-(U2-SCLK-Pad6)
- U2 pad 7: Net-(U2-SIO2) -> unconnected-(U2-SIO3-Pad7)
- U2 pad 8: +3.3V -> unconnected-(U2-VDD-Pad8)
- U3 pad 1: +3.3V -> +3V3
- U3 pad 10: unconnected-(U3-PA2-Pad10) -> /CS2
- U3 pad 11: unconnected-(U3-PA3-Pad11) -> /CS3
- U3 pad 12: Net-(U3-PA4) -> /CS4
- U3 pad 13: Net-(U3-PA5) -> unconnected-(U3-PA5-Pad13)
- U3 pad 14: Net-(U3-PA6) -> unconnected-(U3-PA6-Pad14)
- U3 pad 15: Net-(U3-PA7) -> unconnected-(U3-PA7-Pad15)
- U3 pad 21: Net-(U3-VDDA) -> +3V3
- U3 pad 24: +3.3V -> +3V3
- U3 pad 26: Net-(U2-~{CE}) -> unconnected-(U3-PB12-Pad26)
- U3 pad 27: Net-(U2-SCLK) -> unconnected-(U3-PB13-Pad27)
- U3 pad 28: Net-(U2-SO/SIO1) -> unconnected-(U3-PB14-Pad28)
- U3 pad 29: Net-(U2-SI/SIO0) -> unconnected-(U3-PB15-Pad29)
- U3 pad 32: Net-(U3-PA10) -> unconnected-(U3-PA10-Pad32)
- U3 pad 33: Net-(U3-PA11) -> unconnected-(U3-PA11-Pad33)
- U3 pad 34: Net-(U3-PA12) -> unconnected-(U3-PA12-Pad34)
- U3 pad 36: +3.3V -> +3V3
- U3 pad 37: Net-(U1-INT2) -> unconnected-(U3-PA13-Pad37)
- U3 pad 38: Net-(U1-INT1) -> unconnected-(U3-PA14-Pad38)
- U3 pad 39: Net-(U1-CS) -> unconnected-(U3-PA15-Pad39)
- U3 pad 40: Net-(U1-SDO) -> unconnected-(U3-PB3-Pad40)
- U3 pad 41: Net-(U1-SDI) -> unconnected-(U3-PB4-Pad41)
- U3 pad 42: Net-(U1-SPC) -> unconnected-(U3-PB5-Pad42)
- U3 pad 48: +3.3V -> +3V3
- U3 pad 8: unconnected-(U3-PA0-Pad8) -> /CS0
- U3 pad 9: unconnected-(U3-PA1-Pad9) -> /CS1
- U4 pad 1: Net-(U3-PA4) -> unconnected-(U4-~{CS}-Pad1)
- U4 pad 2: Net-(U3-PA6) -> unconnected-(U4-DO/IO_{1}-Pad2)
- U4 pad 3: Net-(U4-~{HOLD}/~{RESET}/IO_{3}) -> unconnected-(U4-~{WP}/IO_{2}-Pad3)
- U4 pad 5: Net-(U3-PA7) -> unconnected-(U4-DI/IO_{0}-Pad5)
- U4 pad 6: Net-(U3-PA5) -> unconnected-(U4-CLK-Pad6)
- U4 pad 7: Net-(U4-~{HOLD}/~{RESET}/IO_{3}) -> unconnected-(U4-~{HOLD}/~{RESET}/IO_{3}-Pad7)
- U4 pad 8: +3.3V -> unconnected-(U4-VCC-Pad8)
- U5 pad 2: GND -> unconnected-(U5-GND-Pad2)
- U5 pad 3: Net-(U3-PA12) -> unconnected-(U5-~{CS}-Pad3)
- U5 pad 6: Net-(U3-PA11) -> unconnected-(U5-MOSI-Pad6)
- U5 pad 9: Net-(U3-PA10) -> unconnected-(U5-MISO-Pad9)
- U7 pad 1: unconnected-(U7-A-Pad1) -> /SPI1_NSS
- U7 pad 2: unconnected-(U7-B-Pad2) -> /SPI2_NSS
Other:
- copper layers 2 -> 6
- rule pad_to_mask_clearance: 0 -> 0.03

Commit message: refresh
Parts:
- removed U7: 74LVC1G139, Package_SO:VSSOP-8_2.3x2mm_P0.5mm
- C10, C11, C12, C13, C14, C15, C16, C6, C7, C8, C9, U1: moved to B.Cu
- moved H1 63.0 mm to (100.5, 76.5)
- moved H2 59.2 mm to (195.7, 76.4)
- moved H4 52.5 mm to (100.5, 121.6)
- moved U5 48.1 mm to (130.9, 88.9)
- moved H3 43.0 mm to (195.7, 121.6)
- moved U2 29.2 mm to (104.5, 106.6)
- moved J2 26.7 mm to (113.0, 83.0), turned to 180 degrees
- moved C16 21.5 mm to (180.0, 101.6)
- moved C13 21.5 mm to (177.1, 101.6)
- moved C9 21.5 mm to (174.3, 101.6)
- moved U1 21.1 mm to (147.9, 99.0), turned to 180 degrees
- moved J1 19.5 mm to (108.5, 115.7)
- moved C15 19.4 mm to (180.0, 103.5)
- moved C12 19.4 mm to (177.1, 103.5)
- moved C7 19.4 mm to (174.3, 103.5)
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Connections:
- J2 pad 1: unconnected-(J2-DAT2-Pad1) -> Net-(J2-DAT1)
- J2 pad 10: unconnected-(J2-DET_A-Pad10) -> /DET_A
- J2 pad 2: unconnected-(J2-DAT3/CD-Pad2) -> /CS4
- J2 pad 3: unconnected-(J2-CMD-Pad3) -> /SPI_MOSI
- J2 pad 4: unconnected-(J2-VDD-Pad4) -> +3V3
- J2 pad 5: unconnected-(J2-CLK-Pad5) -> /SPI_SCK
- J2 pad 6: unconnected-(J2-VSS-Pad6) -> GND
- J2 pad 7: unconnected-(J2-DAT0-Pad7) -> /SPI_MISO
- J2 pad 8: unconnected-(J2-DAT1-Pad8) -> Net-(J2-DAT1)
- J2 pad 9: unconnected-(J2-DET_B-Pad9) -> GND
- J2 pad SH: unconnected-(J2-SHIELD-PadSH) -> GND
- U1 pad 1: unconnected-(U1-SDO-Pad1) -> /SPI_MISO
- U1 pad 12: unconnected-(U1-CS-Pad12) -> /CS1
- U1 pad 13: unconnected-(U1-SPC-Pad13) -> /SPI_SCK
- U1 pad 14: unconnected-(U1-SDI-Pad14) -> /SPI_MOSI
- U1 pad 2: Net-(U1-GND-Pad2) -> GND
- U1 pad 3: Net-(U1-GND-Pad2) -> GND
- U1 pad 4: unconnected-(U1-INT1-Pad4) -> /EXT1
- U1 pad 5: Net-(U1-VDD) -> +3V3
- U1 pad 6: Net-(U1-GND-Pad2) -> GND
- U1 pad 7: Net-(U1-GND-Pad2) -> GND
- U1 pad 8: Net-(U1-VDD) -> +3V3
- U1 pad 9: unconnected-(U1-INT2-Pad9) -> /EXT2
- U2 pad 1: unconnected-(U2-~{CE}-Pad1) -> /CS2
- U2 pad 2: unconnected-(U2-SO/SIO1-Pad2) -> /SPI_MISO
- U2 pad 3: unconnected-(U2-SIO2-Pad3) -> Net-(U2-SIO2)
- U2 pad 5: unconnected-(U2-SI/SIO0-Pad5) -> /SPI_MOSI
- U2 pad 6: unconnected-(U2-SCLK-Pad6) -> /SPI_SCK
- U2 pad 7: unconnected-(U2-SIO3-Pad7) -> Net-(U2-SIO2)
- U2 pad 8: unconnected-(U2-VDD-Pad8) -> +3V3
- U3 pad 13: unconnected-(U3-PA5-Pad13) -> /SPI_SCK
- U3 pad 14: unconnected-(U3-PA6-Pad14) -> /SPI_MISO
- U3 pad 15: unconnected-(U3-PA7-Pad15) -> /SPI_MOSI
- U3 pad 17: unconnected-(U3-PB1-Pad17) -> /EXT1
- U3 pad 18: unconnected-(U3-PB2-Pad18) -> /EXT2
- U3 pad 22: unconnected-(U3-PB10-Pad22) -> /D/~{C}
- U3 pad 25: unconnected-(U3-PB11-Pad25) -> /DET_A
- U3 pad 26: unconnected-(U3-PB12-Pad26) -> /DET_B
- U4 pad 1: unconnected-(U4-~{CS}-Pad1) -> /CS0
- U4 pad 2: unconnected-(U4-DO/IO_{1}-Pad2) -> /SPI_MISO
- U4 pad 3: unconnected-(U4-~{WP}/IO_{2}-Pad3) -> Net-(U4-~{HOLD}/~{RESET}/IO_{3})
- U4 pad 5: unconnected-(U4-DI/IO_{0}-Pad5) -> /SPI_MOSI
- U4 pad 6: unconnected-(U4-CLK-Pad6) -> /SPI_SCK
- U4 pad 7: unconnected-(U4-~{HOLD}/~{RESET}/IO_{3}-Pad7) -> Net-(U4-~{HOLD}/~{RESET}/IO_{3})
- U4 pad 8: unconnected-(U4-VCC-Pad8) -> +3V3
- U5 pad 1: unconnected-(U5-VCC-Pad1) -> +3V3
- U5 pad 2: unconnected-(U5-GND-Pad2) -> GND
- U5 pad 3: unconnected-(U5-~{CS}-Pad3) -> /CS3
- U5 pad 5: unconnected-(U5-D/~{C}-Pad5) -> /D/~{C}
- U5 pad 6: unconnected-(U5-MOSI-Pad6) -> /SPI_MOSI
- U5 pad 7: unconnected-(U5-SCK-Pad7) -> /SPI_SCK
- U5 pad 8: unconnected-(U5-LED-Pad8) -> +3V3
- U5 pad 9: unconnected-(U5-MISO-Pad9) -> /SPI_MISO
Other:
- board outline added: 100 x 50 mm

Commit message: refresh
Parts:
- added C1: C_Polarized, Capacitor_Tantalum_SMD:CP_EIA-3528-12_Kemet-T, F.Cu at (78.5, 135.7)
- added C2: C_Polarized, Capacitor_Tantalum_SMD:CP_EIA-3528-12_Kemet-T, F.Cu at (78.5, 140.0)
- added C3: C_Polarized, Capacitor_Tantalum_SMD:CP_EIA-3528-12_Kemet-T, F.Cu at (78.5, 144.4)
- added C4: C_Polarized, Capacitor_Tantalum_SMD:CP_EIA-3528-12_Kemet-T, F.Cu at (78.5, 148.7)
- C10, C8: moved to F.Cu
- moved C6 55.1 mm to (124.0, 83.0)
- moved C12 54.6 mm to (124.0, 116.0)
- moved C9 50.3 mm to (124.0, 99.5)
- moved C8 44.6 mm to (127.5, 84.5), turned to -90 degrees
- moved C10 36.8 mm to (127.5, 117.5), turned to -90 degrees
- moved C7 26.8 mm to (157.0, 83.0)
- moved C13 24.8 mm to (157.0, 116.0)
- moved C16 23.1 mm to (157.0, 99.5)
- moved C15 22.8 mm to (190.0, 83.0)
- moved C14 14.5 mm to (190.0, 116.0)
- moved C11 14.2 mm to (190.0, 99.5)
- moved U2 9.74 mm to (104.0, 96.9)

Commit message: refresh
Parts:
- added L1: L, Inductor_SMD:L_Neosid_SM-PIC0512H, F.Cu at (105.0, 105.0)
- added R1: R_US, Resistor_SMD:R_0402_1005Metric_Pad0.72x0.64mm_HandSolder, F.Cu at (116.2, 112.1)
- added R10: R_US, Resistor_SMD:R_0402_1005Metric_Pad0.72x0.64mm_HandSolder, F.Cu at (119.8, 105.6)
- added R11: R_US, Resistor_SMD:R_0402_1005Metric_Pad0.72x0.64mm_HandSolder, F.Cu at (120.7, 105.6)
- added R2: R_US, Resistor_SMD:R_0402_1005Metric_Pad0.72x0.64mm_HandSolder, F.Cu at (108.5, 95.7)
- added R3: R_US, Resistor_SMD:R_0402_1005Metric_Pad0.72x0.64mm_HandSolder, F.Cu at (118.5, 92.9)
- added R4: R_US, Resistor_SMD:R_0402_1005Metric_Pad0.72x0.64mm_HandSolder, F.Cu at (116.2, 109.6)
- added R5: R_US, Resistor_SMD:R_0402_1005Metric_Pad0.72x0.64mm_HandSolder, B.Cu at (147.4, 95.5)
- added R6: R_US, Resistor_SMD:R_0402_1005Metric_Pad0.72x0.64mm_HandSolder, F.Cu at (99.2, 95.6)
- added R7: R_US, Resistor_SMD:R_0402_1005Metric_Pad0.72x0.64mm_HandSolder, F.Cu at (127.9, 94.0)
- added R8: R_US, Resistor_SMD:R_0402_1005Metric_Pad0.72x0.64mm_HandSolder, F.Cu at (111.3, 92.7)
- added R9: R_US, Resistor_SMD:R_0402_1005Metric_Pad0.72x0.64mm_HandSolder, F.Cu at (118.8, 105.6)
- moved C3 52.2 mm to (111.0, 103.5), turned to 90 degrees
- moved C4 49.0 mm to (109.0, 110.4), turned to -90 degrees
- moved C2 37.2 mm to (101.0, 110.4), turned to -90 degrees
- moved C1 29.4 mm to (100.6, 116.4), turned to -90 degrees
- moved C10 9.62 mm to (118.0, 118.8), turned to 90 degrees
- moved U3 6.50 mm to (122.0, 99.0)
- moved U4 0.75 mm to (122.2, 111.5)
Connections:
- C1 pad 2: Net-(U6-GND) -> GND
- C2 pad 2: Net-(U6-GND) -> GND
- C3 pad 1: +3.3V -> +3V3
- C3 pad 2: Net-(U6-GND) -> GND
- C4 pad 2: Net-(U6-GND) -> GND
- J1 pad 2: Net-(U6-GND) -> GND
- J1 pad 3: Net-(U6-GND) -> GND
- U3 pad 10: /CS2 -> Net-(U3-PA2)
- U3 pad 11: /CS3 -> Net-(U3-PA3)
- U3 pad 12: /CS4 -> Net-(U3-PA4)
- U3 pad 13: /SPI_SCK -> Net-(U3-PA5)
- U3 pad 14: /SPI_MISO -> Net-(U3-PA6)
- U3 pad 15: /SPI_MOSI -> Net-(U3-PA7)
- U3 pad 8: /CS0 -> Net-(U3-PA0)
- U3 pad 9: /CS1 -> Net-(U3-PA1)
- U6 pad 2: Net-(U6-GND) -> GND
Routing:
- net /SPI_MOSI: track 0.00 -> 52.2 mm, vias 0 -> 2
- net /SPI_SCK: track 0.00 -> 45.9 mm, vias 0 -> 1
- net /EXT1: track 0.00 -> 33.6 mm, vias 0 -> 1
- net Net-(U3-PA1): track 0.00 -> 31.1 mm, vias 0 -> 2
- net /EXT2: track 0.00 -> 27.8 mm, vias 0 -> 1
- net /SPI_MISO: track 0.00 -> 25.1 mm, vias 0 -> 1
- net +5V: track 0.00 -> 22.7 mm
- net Net-(U3-PA2): track 0.00 -> 21.8 mm, vias 0 -> 2
- net Net-(U6-VOUT): track 0.00 -> 17.7 mm
- net Net-(U3-PA4): track 0.00 -> 12.7 mm, vias 0 -> 2
- net Net-(U3-PA3): track 0.00 -> 12.2 mm
- net Net-(U3-PA0): track 0.00 -> 11.6 mm
- net +3V3: track 0.00 -> 7.60 mm, vias 0 -> 6
- net /CS3: track 0.00 -> 2.35 mm
- net /CS2: track 0.00 -> 2.33 mm
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- added copper zone on In3.Cu, net +3V3

Commit message: refresh
Routing:
- net /SPI_MISO: track 25.1 -> 81.1 mm
- net /SPI_SCK: track 45.9 -> 66.5 mm
- net /SPI_MOSI: track 52.2 -> 70.0 mm
- net +3V3: track 7.60 -> 25.3 mm, vias 6 -> 7
- net /D/~{C}: track 0.00 -> 10.4 mm
- net Net-(J2-DAT1): track 2.19 -> 10.5 mm, vias 0 -> 2
- net Net-(U2-SIO2): track 2.03 -> 7.41 mm
