File: Gyroscope.kicad_pcb (KiCad board)
At the start: 6 copper layers, 100 x 50 mm, 39 parts, among them J1 Barrel_Jack_Switch, J2 Micro_SD_Card_Det2, U1 IIS3DWB, U2 APS6404L-3SQRx-SN, U3 STM32G431C6Tx, U4 W25Q128JVS, U5 CR2013-MI2120, U6 AP2112K-3.3

Commit message: refresh
Parts:
- turned C6 to 180 degrees
Routing:
- net /SPI_MISO: track 81.1 -> 116.2 mm, vias 1 -> 2
- net /SPI_MOSI: track 70.0 -> 98.6 mm, vias 2 -> 3
- net /DET_A: track 0.00 -> 27.2 mm, vias 0 -> 2
- net /SPI_SCK: track 66.5 -> 92.9 mm, vias 1 -> 4
- net GND: track 0.00 -> 24.7 mm, vias 0 -> 138
- net Net-(U4-~{HOLD}/~{RESET}/IO_{3}): track 1.86 -> 9.37 mm
- net +3V3: track 25.3 -> 27.9 mm, vias 7 -> 22
- added copper zone on B.Cu, net GND
- added copper zone on F.Cu, net GND
- added copper zone on In1.Cu, net GND
- added copper zone on In2.Cu, net GND
- added copper zone on In4.Cu, net GND
