File: Gyroscope.kicad_sch (KiCad schematic)
At the start: 1 part, among them U1 ADXL343

Commit message: refresh
Parts:
- removed U1: ADXL343, Package_LGA:LGA-14_3x5mm_P0.8mm_LayoutBorder1x6y, symbol Sensor_Motion:ADXL343
- added C1, C2, C3, C4: C_Polarized, symbol Device:C_Polarized
- added FB1: FerriteBead, symbol Device:FerriteBead
- added J1: Barrel_Jack_Switch, symbol Connector:Barrel_Jack_Switch
- added L1: L, symbol Device:L
- added U1: IIS3DWB, Package_LGA:LGA-14_3x2.5mm_P0.5mm_LayoutBorder3x4y, symbol Sensor_Motion:IIS3DWB
- added U2: APS6404L-3SQRx-SN, Package_SO:SOIC-8_3.9x4.9mm_P1.27mm, symbol Memory_RAM:APS6404L-3SQRx-SN
- added U3: STM32G431C6Tx, Package_QFP:LQFP-48_7x7mm_P0.5mm, symbol MCU_ST_STM32G4:STM32G431C6Tx
- added U4: W25Q128JVS, Package_SO:SOIC-8_5.3x5.3mm_P1.27mm, symbol Memory_Flash:W25Q128JVS
- added U5: CR2013-MI2120, Display:CR2013-MI2120, symbol Driver_Display:CR2013-MI2120
- added U6: AP2112K-3.3, Package_TO_SOT_SMD:SOT-23-5, symbol Regulator_Linear:AP2112K-3.3
Connections:
- new net: FB1.1, U3.1 (VBAT), U3.24 (VDD), U3.36 (VDD), U3.48 (VDD)
- new net: FB1.2, U3.21 (VDDA)
- new net: C2.1, C4.1, L1.1, U6.5 (VOUT)
- new net: C1.2, C2.2, C3.2, C4.2, J1.2, J1.3, U6.2 (GND)
- new net +3.3V: C3.1, L1.2
- new net +5V: C1.1, J1.1, U6.1 (VIN), U6.3 (EN)
- new net GND: U1.2 (GND), U1.3 (GND), U1.6 (GND), U1.7 (GND), U2.4 (VSS), U3.19 (VSSA), U3.23 (VSS), U3.35 (VSS), U3.47 (VSS), U4.4 (GND), U5.2 (GND)

Commit message: refresh
Parts:
- added J2: Micro_SD_Card_Det2, Connector_Card:microSD_HC_Hirose_DM3AT-SF-PEJM5, symbol Connector:Micro_SD_Card_Det2
- added R1, R2: R_US, symbol Device:R_US
Connections:
- net +3.3V: now also FB1.1, U2.8 (VDD), U3.1 (VBAT), U3.24 (VDD), U3.36 (VDD), U3.48 (VDD), U4.8 (VCC), R1.1, R2.1
- net at U5.3 (~{CS}): now also U3.34 (PA12)
- net at U5.6 (MOSI): now also U3.33 (PA11)
- net at U5.9 (MISO): now also U3.32 (PA10)
- net at U2.1 (~{CE}): now also U3.26 (PB12)
- net at U2.2 (SO/SIO1): now also U3.28 (PB14)
- net at U2.3 (SIO2): now also U2.7 (SIO3), R2.2
- net at U2.5 (SI/SIO0): now also U3.29 (PB15)
- net at U2.6 (SCLK): now also U3.27 (PB13)
- net at U3.12 (PA4): now also U4.1 (~{CS})
- net at U3.13 (PA5): now also U4.6 (CLK)
- net at U3.14 (PA6): now also U4.2 (DO/IO_{1})
- net at U3.15 (PA7): now also U4.5 (DI/IO_{0})
- net at U3.37 (PA13): now also U1.9 (INT2)
- net at U3.38 (PA14): now also U1.4 (INT1)
- net at U3.39 (PA15): now also U1.12 (CS)
- net at U3.40 (PB3): now also U1.1 (SDO)
- net at U3.41 (PB4): now also U1.14 (SDI)
- net at U3.42 (PB5): now also U1.13 (SPC)
- net at U4.3 (~{WP}/IO_{2}): now also U4.7 (~{HOLD}/~{RESET}/IO_{3}), R1.2
- net at U1.5 (VDD_IO): now also U1.8 (VDD)
Other:
- moved on the sheet: FB1, U1, U2, U4, U5

Commit message: refresh
Parts:
- added H1, H2, H3, H4: MountingScrew, MountingHole:MountingHole_2.2mm_M2_DIN965_Pad_TopBottom, symbol Auxiliary_Items:MountingScrew
- added U7: 74LVC1G139, Package_SO:VSSOP-8_2.3x2mm_P0.5mm, symbol 74xGxx:74LVC1G139
- J1: footprint (none) -> Connector_BarrelJack:BarrelJack_GCT_DCJ200-10-A_Horizontal
Connections:
- net +3.3V: no longer U4.8 (VCC)
- net at U5.3 (~{CS}): no longer U3.34 (PA12)
- net at U5.6 (MOSI): no longer U3.33 (PA11)
- net at U5.9 (MISO): no longer U3.32 (PA10)
- net at U2.1 (~{CE}): no longer U3.26 (PB12)
- net at U2.2 (SO/SIO1): no longer U3.28 (PB14)
- net at U2.5 (SI/SIO0): no longer U3.29 (PB15)
- net at U2.6 (SCLK): no longer U3.27 (PB13)
- net at U3.12 (PA4): no longer U4.1 (~{CS})
- net at U3.13 (PA5): no longer U4.6 (CLK)
- net at U3.14 (PA6): no longer U4.2 (DO/IO_{1})
- net at U3.15 (PA7): no longer U4.5 (DI/IO_{0})
- net at U3.37 (PA13): no longer U1.9 (INT2)
- net at U3.38 (PA14): no longer U1.4 (INT1)
- net at U3.39 (PA15): no longer U1.12 (CS)
- net at U3.40 (PB3): no longer U1.1 (SDO)
- net at U3.41 (PB4): no longer U1.14 (SDI)
- net at U3.42 (PB5): no longer U1.13 (SPC)
- now unconnected: R1.2, R2.2, U2.3 (SIO2), U2.7 (SIO3), U4.3 (~{WP}/IO_{2}), U4.7 (~{HOLD}/~{RESET}/IO_{3})
Other:
- moved on the sheet: C1, C2, C3, C4, J1, L1, U6

Commit message: refresh
Parts:
- removed FB1: FerriteBead, symbol Device:FerriteBead
- removed R1, R2: R_US, symbol Device:R_US
- added C10, C8: 1u, Capacitor_SMD:C_0805_2012Metric, symbol Device:C
- added C11, C12, C13, C14, C15, C16, C6, C7, C9: 100n, Capacitor_SMD:C_0402_1005Metric, symbol Device:C_Small
Connections:
- net +3.3V: no longer U2.8 (VDD), U3.1 (VBAT), U3.24 (VDD), U3.36 (VDD), U3.48 (VDD)
- net GND: now also C10.1, C11.2, C12.2, C13.2, C14.2, C15.2, C16.2, C6.2, C7.2, C8.1, C9.2; no longer U1.2 (GND), U1.3 (GND), U1.6 (GND), U1.7 (GND), U2.4 (VSS), U5.2 (GND)
- net CS2: now reaches U3.10 (PA2)
- net CS3: now reaches U3.11 (PA3)
- net CS4: now reaches U3.12 (PA4)
- net +3V3: now reaches U3.21 (VDDA)
- net +3V3: now also U3.1 (VBAT), U3.24 (VDD), U3.36 (VDD), U3.48 (VDD), C10.2, C11.1, C12.1, C13.1, C14.1, C15.1, C16.1, C6.1, C7.1, C8.2, C9.1
- net CS0: now reaches U3.8 (PA0)
- net CS1: now reaches U3.9 (PA1)
- net SPI1_NSS: now reaches U7.1 (A)
- net SPI2_NSS: now reaches U7.2 (B)
- new net: U1.2 (GND), U1.3 (GND), U1.6 (GND), U1.7 (GND)
Other:
- moved on the sheet: C1, C2, C3, C4, J1, L1, U6, U7

Commit message: refresh
Parts:
- removed U7: 74LVC1G139, Package_SO:VSSOP-8_2.3x2mm_P0.5mm, symbol 74xGxx:74LVC1G139
- added R1, R2, R3: R_US, symbol Device:R_US
Connections:
- net +3V3: now also J2.4 (VDD), U1.5 (VDD_IO), U1.8 (VDD), U2.8 (VDD), U4.8 (VCC), U5.1 (VCC), U5.8 (LED), R1.1, R2.2, R3.1
- net CS0: now also U4.1 (~{CS})
- net CS1: now also U1.12 (CS)
- net CS2: now also U2.1 (~{CE})
- net CS3: now also U5.3 (~{CS})
- net CS4: now also J2.2 (DAT3/CD)
- net GND: now also J2.6 (VSS), J2.9 (DET_B), J2.SH (SHIELD), U1.2 (GND), U1.3 (GND), U1.6 (GND), U1.7 (GND), U5.2 (GND)
- net D/~{C}: now reaches U5.5 (D/~{C})
- net D/~{C}: now also U3.22 (PB10)
- net SPI_MOSI: now reaches U5.6 (MOSI)
- net SPI_MOSI: now also J2.3 (CMD), U1.14 (SDI), U2.5 (SI/SIO0), U3.15 (PA7), U4.5 (DI/IO_{0})
- net SPI_SCK: now reaches U5.7 (SCK)
- net SPI_SCK: now also J2.5 (CLK), U1.13 (SPC), U2.6 (SCLK), U3.13 (PA5), U4.6 (CLK)
- net SPI_MISO: now reaches U5.9 (MISO)
- net SPI_MISO: now also J2.7 (DAT0), U1.1 (SDO), U2.2 (SO/SIO1), U3.14 (PA6), U4.2 (DO/IO_{1})
- net at U2.3 (SIO2): now also U2.7 (SIO3), R2.1
- net EXT1: now reaches U3.17 (PB1)
- net EXT1: now also U1.4 (INT1)
- net EXT2: now reaches U3.18 (PB2)
- net EXT2: now also U1.9 (INT2)
- net DET_A: now reaches U3.25 (PB11)
- net DET_A: now also J2.10 (DET_A)
- net DET_B: now reaches U3.26 (PB12)
- net at U4.3 (~{WP}/IO_{2}): now also U4.7 (~{HOLD}/~{RESET}/IO_{3}), R1.2
- net at J2.1 (DAT2): now also J2.8 (DAT1), R3.2
- no-connect marks 0 -> 6
Other:
- moved on the sheet: C10, C11, C12, C13, C14, C15, C16, C6, C7, C8, C9, J2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

Commit message: refresh
Parts:
- C1, C2, C3, C4: footprint (none) -> Capacitor_Tantalum_SMD:CP_EIA-3528-12_Kemet-T
Changed lines of the file:
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@@
 			)
 		)
-		(property "Footprint" ""
+		(property "Footprint" "Capacitor_Tantalum_SMD:CP_EIA-3528-12_Kemet-T"
 			(at 40.3352 30.48 0)
 			(hide yes)
@@
 			)
 		)
-		(property "Footprint" ""
+		(property "Footprint" "Capacitor_Tantalum_SMD:CP_EIA-3528-12_Kemet-T"
 			(at 110.1852 30.48 0)
 			(hide yes)
@@
 			)
 		)
-		(property "Footprint" ""
+		(property "Footprint" "Capacitor_Tantalum_SMD:CP_EIA-3528-12_Kemet-T"
 			(at 91.1352 30.48 0)
 			(hide yes)
@@
 			)
 		)
-		(property "Footprint" ""
+		(property "Footprint" "Capacitor_Tantalum_SMD:CP_EIA-3528-12_Kemet-T"
 			(at 135.5852 30.48 0)
 			(hide yes)

Commit message: refresh
Parts:
- added R10, R11, R4, R5, R6, R7, R8, R9: R_US, Resistor_SMD:R_0402_1005Metric_Pad0.72x0.64mm_HandSolder, symbol Device:R_US
- L1: footprint (none) -> Inductor_SMD:L_Neosid_SM-PIC0512H
- R1, R2, R3: footprint (none) -> Resistor_SMD:R_0402_1005Metric_Pad0.72x0.64mm_HandSolder
Connections:
- net +3.3V is gone; now on net +3V3: C3.1, L1.2
- net CS0: now also R4.1; no longer U3.8 (PA0)
- net CS1: now also R5.1; no longer U3.9 (PA1)
- net CS2: now also R6.1; no longer U3.10 (PA2)
- net CS3: now also R7.1; no longer U3.11 (PA3)
- net CS4: now also R8.1; no longer U3.12 (PA4)
- net GND: now also C1.2, C2.2, C3.2, C4.2, J1.2, J1.3, U6.2 (GND)
- net SPI_MISO: now also R10.1; no longer U3.14 (PA6)
- net SPI_MOSI: now also R11.1; no longer U3.15 (PA7)
- net SPI_SCK: now also R9.1; no longer U3.13 (PA5)
- new net: R11.2, U3.15 (PA7)
- new net: R6.2, U3.10 (PA2)
- new net: R7.2, U3.11 (PA3)
- new net: R8.2, U3.12 (PA4)
- new net: R9.2, U3.13 (PA5)
- new net: R10.2, U3.14 (PA6)
- new net: R4.2, U3.8 (PA0)
- new net: R5.2, U3.9 (PA1)
Other:
- moved on the sheet: C10, C11, C12, C13, C14, C15, C16, C6, C7, C8, C9, U3

Commit message: refresh
Other:
- company: (none) -> IslamHUFE
- title: (none) -> Mechanical vibrations monitor
Changed lines of the file:
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@@
 	(generator_version "10.0")
 	(paper "A4")
+	(title_block
+		(title "Mechanical vibrations monitor")
+		(date "2026-05-29")
+		(rev "Islam Tarek")
+		(company "IslamHUFE")
+	)
 	(junction
 		(at 39.37 22.86)
