File: Gyroscope.kicad_sch (KiCad schematic)
At the start: 39 parts, among them J1 Barrel_Jack_Switch, J2 Micro_SD_Card_Det2, U1 IIS3DWB, U2 APS6404L-3SQRx-SN, U3 STM32G431C6Tx, U4 W25Q128JVS, U5 CR2013-MI2120, U6 AP2112K-3.3

Commit message: refresh
Other:
- note added: "DECOUBLING CAPACITORS"
- note added: "MAIN MEMORY"
- note added: "MCU"
- note added: "MONITOR"
- note added: "MOUNTING SCREWS"
- note added: "POWER"
- note added: "SECOUNDRY MEMORY"
- note added: "SENSOR"
- moved on the sheet: C1, C10, C11, C12, C13, C14, C15, C16, C2, C3, C4, C6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
